File: hardware/test_platform/test_platform.kicad_sch (KiCad schematic)
At the start: 136 parts

Commit message: success initialization of SST25V040 flash memory
Parts:
- removed PAD2: (no value), symbol centralaV2.2-eagle-import:1,6/0,8
- C1, C10, C11, C12, C13, C3, C4, C7: value (none) -> 100n; footprint (none) -> centralaV2.2:C0805
- C14: value (none) -> 33n; footprint (none) -> centralaV2.2:C0805
- C2, C6: value (none) -> 100u; footprint (none) -> centralaV2.2:E2,5-7
- C5: value (none) -> 100u/25V; footprint (none) -> centralaV2.2:E2,5-7
- C8: value (none) -> 22u; footprint (none) -> centralaV2.2:SMC_D
- C9: value (none) -> 22p; footprint (none) -> centralaV2.2:C0805
- CON1, CON2: value (none) -> CON10; footprint (none) -> centralaV2.2:CON10
- D1, D2: value (none) -> PMLL41SOD80C; footprint (none) -> centralaV2.2:SOD80C
- D10, D11, D12, D8, D9: value (none) -> SFH482; footprint (none) -> centralaV2.2:SFH482
- D13, D14, D15, D6, D7: value (none) -> 1N4148; footprint (none) -> centralaV2.2:SOD80C
- D4, D5: value (none) -> 3V6; footprint (none) -> centralaV2.2:SOD80C
- F1, F2, F3, F5: value (none) -> 1A; footprint (none) -> centralaV2.2:CT_CN1812
- F4: value (none) -> 0.5A; footprint (none) -> centralaV2.2:CT_CN1812
- IC1: value (none) -> TS2940; footprint (none) -> centralaV2.2:TO220V
- IC2: value (none) -> LTC485S; footprint (none) -> centralaV2.2:SOIC8
- IC3: value (none) -> PFC8583T; footprint (none) -> centralaV2.2:SO8-7_5
- IC4: value (none) -> PIC18F6J50; footprint (none) -> centralaV2.2:TQFP64-10X10
- IC5: value (none) -> 78DT; footprint (none) -> centralaV2.2:TO252
- IC6: value (none) -> 24SM; footprint (none) -> centralaV2.2:SO-08M
- IC7: value (none) -> FT232RL; footprint (none) -> centralaV2.2:SSOP28
- J1: value (none) -> MTA02-100; footprint (none) -> centralaV2.2:10X02MTA
- J10, J6, J7, J9: value (none) -> MTA03-156; footprint (none) -> centralaV2.2:1X3MTA
- J2: value (none) -> MTA05-100; footprint (none) -> centralaV2.2:10X05MTA
- J3: value (none) -> MTA03-100; footprint (none) -> centralaV2.2:10X03MTA
- J4, J5: value (none) -> MTA10-100; footprint (none) -> centralaV2.2:10X10MTA
- J8: value (none) -> MTA04-100; footprint (none) -> centralaV2.2:10X04MTA
- K1: value (none) -> FTR-F1CA012V; footprint (none) -> centralaV2.2:G2R2
- K2, K3: footprint (none) -> centralaV2.2:G2R2
- LED3, LED4: value (none) -> LEDCHIP-LED0805; footprint (none) -> centralaV2.2:CHIP-LED0805
- Q1, Q2, Q3, Q4, Q5: value (none) -> BC817; footprint (none) -> centralaV2.2:SOT23-BEC
- R1, R10, R12, R2, R27, R29, R3, R34, R35: value (none) -> 200R; footprint (none) -> centralaV2.2:R0805
- R11, R17, R19, R28, R30, R32, R33, R36, R37, R38, R4, R41, R42, R43, R47, R49, R5, R51, R6, R7: value (none) -> 10k; footprint (none) -> centralaV2.2:R0805
- R13: value (none) -> 10k; footprint (none) -> centralaV2.2:RTRIM3299W
- R14, R16, R46, R48, R50: value (none) -> 4,7k; footprint (none) -> centralaV2.2:R0805
- R15, R21, R24, R25, R39, R40: value (none) -> 1k; footprint (none) -> centralaV2.2:R0805
- R18: value (none) -> 10uH/450mA; footprint (none) -> centralaV2.2:M1206
- R20, R22: value (none) -> 18k; footprint (none) -> centralaV2.2:R0805
- R23, R26: value (none) -> 240R; footprint (none) -> centralaV2.2:R0805
- R52, R53, R54: value (none) -> S20K250; footprint (none) -> centralaV2.2:S20K250
- R8: value (none) -> 620R; footprint (none) -> centralaV2.2:R0805
- R9: value (none) -> 2.2k; footprint (none) -> centralaV2.2:R0805
- S1, S2, S3: value (none) -> 40-XX; footprint (none) -> centralaV2.2:B3F_40XXA
- T1, T2, T3, T4: value (none) -> -PNP-SOT23-BEC; footprint (none) -> centralaV2.2:SOT23-BEC
- TR1, TR2: value (none) -> TGL34-6.8CA; footprint (none) -> centralaV2.2:DO214AC+MINIMELF_BIDIR
- U$1: value (none) -> SST25VF016B; footprint (none) -> centralaV2.2:SOIC8(S2A)
- U$10: value (none) -> 5PIN_R2,54; footprint (none) -> centralaV2.2:5PIN_R2,54
- U$11: value (none) -> CR2032; footprint (none) -> centralaV2.2:CR2032
- U$12: value (none) -> RG12864B-BIW-V; footprint (none) -> centralaV2.2:RG12864B-BIW-V
- U$2: value (none) -> AMSR-7815-NZ; footprint (none) -> centralaV2.2:AIMTEC_DC
- U$3: value (none) -> USBB; footprint (none) -> centralaV2.2:USB_B
- U$4, U$5: value (none) -> TXB010X; footprint (none) -> centralaV2.2:TSSOP20
- U$6: value (none) -> G5Q; footprint (none) -> centralaV2.2:G5Q_SPSTNO
- U$7: value (none) -> XL4015; footprint (none) -> centralaV2.2:DC_BUCK
- U$8: value (none) -> 4PIN_R3,96; footprint (none) -> centralaV2.2:4PIN_R3,96
- U$9: value (none) -> 3PIN_R3,96; footprint (none) -> centralaV2.2:3PIN_R3,96
- Y1: value (none) -> 32.768kHz; footprint (none) -> centralaV2.2:CRYSTAL-PTH-2X6-CYL-KIT
Connections:
- net ALARM_RLY: no longer IC4.35 (RC4/SDI1/SDA1)
- net MAIN_SPL_RLY: no longer IC4.34 (RC3/SCK1/SCL1)
- net RC5: no longer IC4.36 (RC5/SDO1/C2OUT)
- net SOFT_RLY: no longer IC4.33 (RC2/ECCP1/P1A)
- net SST25_CLK: now also IC4.34 (RC3/SCK1/SCL1); no longer IC4.46 (RB2/INT2/PMA3)
- net SST25_CS: now also IC4.11 (RF7/~{SS1}/C1OUT); no longer IC4.43 (RB5/KBI1/PMA0)
- net SST25_DI: now also IC4.35 (RC4/SDI1/SDA1); no longer IC4.45 (RB3/INT3/PMA2)
- net SST25_DO: now also IC4.36 (RC5/SDO1/C2OUT); no longer IC4.44 (RB4/KBI0/PMA1)
