File: hardware/battery_tester_v1.0/battery_tester_v1.0/battery_tester_v1.0.kicad_sch (KiCad schematic)
At the start: 0 parts

Commit message: update battery tester
Other:
- added sheet Current Source (current_source.kicad_sch)
Changed lines of the file:
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@@
 	(paper "A4")
+	(sheet
+		(at 84.074 25.908)
+		(size 34.29 31.242)
+		(exclude_from_sim no)
+		(in_bom yes)
+		(on_board yes)
+		(dnp no)
+		(fields_autoplaced yes)
+		(stroke
+			(width 0.1524)
+			(type solid)
+		)
+		(fill
+			(color 0 0 0 0.0000)
+		)
+		(property "Sheetname" "Current Source"
+			(at 84.074 25.1964 0)
+			(effects
+				(font
+					(size 1.27 1.27)
+				)
+				(justify left bottom)
+			)
+		)
+		(property "Sheetfile" "current_source.kicad_sch"
+			(at 84.074 57.7346 0)
+			(effects
+				(font
+					(size 1.27 1.27)
+				)
+				(justify left top)
+			)
+		)
+		(instances
+			(project "battery_tester_v1.0"
+				(path "/3840e110-92c0-43e0-a480-527208a59562"
+					(page "3")
+				)
+			)
+		)
+	)
 	(sheet
 		(at 34.29 25.908)

Commit message: update lcd pcb
Other:
- sheet Microcontroller renamed microcontroller
Changed lines of the file:
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@@
 			(color 0 0 0 0.0000)
 		)
-		(property "Sheetname" "Microcontroller"
+		(property "Sheetname" "microcontroller"
 			(at 34.29 25.1964 0)
 			(effects
