File: hardware/battery_tester_v1.0/battery_tester_v1.0/current_source.kicad_sch (KiCad schematic)
At the start: 13 parts, among them K1 Relay_DPDT, Q1 IRF540N, U1 LM358

Commit message: update lcd pcb
Connections:
- net ADC_DISCHARGE_CURRENT: now reaches R8.1, U1.7
Changed lines of the file:
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@@
 		(color 0 0 0 0)
 	)
+	(junction
+		(at 53.34 87.63)
+		(diameter 0)
+		(color 0 0 0 0)
+	)
 	(wire
 		(pts
@@
 	(wire
 		(pts
+			(xy 45.72 87.63) (xy 53.34 87.63)
+		)
+		(stroke
+			(width 0)
+			(type default)
+		)
+	)
+	(wire
+		(pts
 			(xy 90.17 85.09) (xy 90.17 92.71)
 		)
@@
 		)
 	)
+	(global_label "ADC_DISCHARGE_CURRENT"
+		(shape input)
+		(at 45.72 87.63 180)
+		(fields_autoplaced yes)
+		(effects
+			(font
+				(size 1.27 1.27)
+			)
+			(justify right)
+		)
+		(property "Intersheetrefs" "${INTERSHEET_REFS}"
+			(at 18.121 87.63 0)
+			(effects
+				(font
+					(size 1.27 1.27)
+				)
+				(justify right)
+				(hide yes)
+			)
+		)
+	)
