File: hardware/128X64 LCD display + 9x button matrix V1.0/20pin_lcd_display.kicad_sch (KiCad schematic)
At the start: 75 parts, among them J1 VCC_5V, J2 LED, J3 LED, Q1 BC817, Q2 BC817, Q3 BC817, Q4 BC817, SW1 SW_Push, SW2 SW_Push, SW3 SW_Push, SW4 SW_Push, SW5 SW_Push, SW6 SW_Push, SW7 SW_Push, SW8 SW_Push, SW9 SW_Push, U1 74AHCT244, U2 74HCT125, U3 74HC595, U4 74HC595

Commit message: update man pcb, cleanup
Other:
- note added: "BUFFERS"
- note added: "CONNECTORS"
- note added: "DIRECT CONNECTION OF LCD"
- note added: "FOR SHIFT REGISTER MODE"
- note added: "LCD CONNECTIONS TYPES: - DIRECT: SOLDER ALL RESISTORS R3-R15 (0R) NO SHIFT REGISTERS AND BUFFERS - BUFFERS: SOLDER ONLY BUFFERS AND R21 RESISTOR (BACKLIGHT) - SHIFT REGISTERS: ONLY SHIFT REGISTERS"
- note added: "M3 MOUTING PADS"
- note added: "PUSH BUTTONS MATRIX"
- note added: "RG12864B-BIW 128x64 LCD DISPLAY"
- note added: "SHIFT REGISTERS"
- note removed: "PUSH BUTTONS"
- moved on the sheet: C6, D1, D10, D11, D12, D2, D3, D4, D5, D6, D7, D8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
