File: hardware/Battery tester V1.0/battery_tester_v1.0.kicad_sch (KiCad schematic)
At the start: 0 parts

Commit message: update man pcb, cleanup
Other:
- sheet microcontroller renamed Microcontroller
- added sheet Charger (charger.kicad_sch)
Changed lines of the file:
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@@
 	(paper "A4")
+	(sheet
+		(at 137.16 25.4)
+		(size 36.83 31.75)
+		(exclude_from_sim no)
+		(in_bom yes)
+		(on_board yes)
+		(dnp no)
+		(fields_autoplaced yes)
+		(stroke
+			(width 0.1524)
+			(type solid)
+		)
+		(fill
+			(color 0 0 0 0.0000)
+		)
+		(property "Sheetname" "Charger"
+			(at 137.16 24.6884 0)
+			(effects
+				(font
+					(size 1.27 1.27)
+				)
+				(justify left bottom)
+			)
+		)
+		(property "Sheetfile" "charger.kicad_sch"
+			(at 137.16 57.7346 0)
+			(effects
+				(font
+					(size 1.27 1.27)
+				)
+				(justify left top)
+			)
+		)
+		(instances
+			(project "battery_tester_v1.0"
+				(path "/3840e110-92c0-43e0-a480-527208a59562"
+					(page "4")
+				)
+			)
+		)
+	)
 	(sheet
 		(at 84.074 25.908)
@@
 			(color 0 0 0 0.0000)
 		)
-		(property "Sheetname" "microcontroller"
+		(property "Sheetname" "Microcontroller"
 			(at 34.29 25.1964 0)
 			(effects
