File: hardware/Battery tester V1.0/charger.kicad_sch (KiCad schematic)
At the start: 0 parts

Commit message: update main pcb schematic
Parts:
- added C14, C20: 100n, Capacitor_SMD:C_0805_2012Metric_Pad1.18x1.45mm_HandSolder, symbol Device:C
- added C15, C19: 1u, Capacitor_SMD:C_0805_2012Metric_Pad1.18x1.45mm_HandSolder, symbol Device:C
- added C16, C17, C18: 470u, symbol Device:C_Polarized
- added D2: D_Schottky, symbol Device:D_Schottky_Dual_CommonCathode_KAA_Parallel
- added L1: 47uH, symbol Device:L
- added U6: XL4015, Package_TO_SOT_SMD:TO-263-5_TabPin3, symbol Regulator_Switching:XL4015
Connections:
- new net: C17.1, C18.1, C19.1, C20.1, L1.2
- new net: C14.2, C16.2, C17.2, C18.2, C19.2, C20.2, D2.2 (K), D2.3 (K), U6.1 (GND)
- new net: D2.1 (A), L1.1, U6.3 (SW)
- new net: C15.2, U6.4 (VC)
- new net VCC: C14.1, C15.1, C16.1, U6.5 (VIN)

Commit message: update main pcb battery charger
Parts:
- added C10, C34, C39, C43: 100p, Capacitor_SMD:C_0805_2012Metric_Pad1.18x1.45mm_HandSolder, symbol Device:C
- added C24, C25, C26, C29, C30, C31 (x2), C32 (x2), C33, C36, C37, C40, C41, C42, C7, C8, C9: 100n, Capacitor_SMD:C_0805_2012Metric_Pad1.18x1.45mm_HandSolder, symbol Device:C
- added C27, C28: 1n, Capacitor_SMD:C_0805_2012Metric_Pad1.18x1.45mm_HandSolder, symbol Device:C
- added C33, C34: 1u, Capacitor_SMD:C_0805_2012Metric_Pad1.18x1.45mm_HandSolder, symbol Device:C
- added C35: 220u/63V, Capacitor_THT:CP_Radial_D10.0mm_P5.00mm, symbol Device:C_Polarized
- added C38: 10u/63V, Capacitor_SMD:C_1206_3216Metric, symbol Device:C
- added D1, D3, D4, D5: 1N4148, Diode_THT:D_DO-35_SOD27_P7.62mm_Horizontal, symbol Diode:1N4148
- added D10, D11, D8, D9: LL4148, Diode_SMD:D_MiniMELF, symbol Diode:LL4148
- added J6: Conn_01x04, symbol Connector_Generic:Conn_01x04
- added K1, K2: Relay_DPDT, symbol Relay:Relay_DPDT
- added Q1, Q3, Q7: BC817, Package_TO_SOT_SMD:SOT-23, symbol Transistor_BJT:BC817
- added Q10: 2SC2655, My-Footprints:TO-92_Inline_LITTLE_BIGGER, symbol Transistor_BJT:SS8050
- added Q2: IRF540N, Package_TO_SOT_THT:TO-220-3_Vertical, symbol Transistor_FET:IRF540N
- added Q8: BD136, Package_TO_SOT_THT:TO-126-3_Vertical, symbol Transistor_BJT:BD136
- added R10, R15, R16, R17, R6, R7: 1k, Capacitor_SMD:C_0805_2012Metric_Pad1.18x1.45mm_HandSolder, symbol Device:R
- added R11: 0R1, Capacitor_SMD:C_0805_2012Metric_Pad1.18x1.45mm_HandSolder, symbol Device:R
- added R12: 1R, Capacitor_SMD:C_0805_2012Metric_Pad1.18x1.45mm_HandSolder, symbol Device:R
- added R18, R19, R8: 10k, Capacitor_SMD:C_0805_2012Metric_Pad1.18x1.45mm_HandSolder, symbol Device:R
- added R20, R23, R24, R25 (x2), R27, R28, R31, R32, R33: 10k, Resistor_SMD:R_0805_2012Metric_Pad1.20x1.40mm_HandSolder, symbol Device:R
- added R21, R22: 470R, Resistor_SMD:R_0805_2012Metric_Pad1.20x1.40mm_HandSolder, symbol Device:R
- added R26, R34, R35, R39, R40, R41, R42, R45, R46: 1k, Resistor_SMD:R_0805_2012Metric_Pad1.20x1.40mm_HandSolder, symbol Device:R
- added R29: 1K, Resistor_SMD:R_0805_2012Metric_Pad1.20x1.40mm_HandSolder, symbol Device:R
- added R30: 2k7, Resistor_SMD:R_0805_2012Metric_Pad1.20x1.40mm_HandSolder, symbol Device:R
- added R38: 10R, Resistor_SMD:R_0805_2012Metric_Pad1.20x1.40mm_HandSolder, symbol Device:R
- added R5: 3k9, Capacitor_SMD:C_0805_2012Metric_Pad1.18x1.45mm_HandSolder, symbol Device:R
- added R9: 100R, Capacitor_SMD:C_0805_2012Metric_Pad1.18x1.45mm_HandSolder, symbol Device:R
- added U10: MCP4725xxx-xCH, Package_TO_SOT_SMD:SOT-23-6, symbol Analog_DAC:MCP4725xxx-xCH
- added U10, U9: OP07, Package_SO:SO-8_3.9x4.9mm_P1.27mm, symbol Amplifier_Operational:OP07
- added U11: LM324, Package_SO:SO-14_3.9x8.65mm_P1.27mm, symbol Amplifier_Operational:LM324
- added U2: LM358, Package_SO:SO-8_3.9x4.9mm_P1.27mm, symbol Amplifier_Operational:LM358
- added U7: LM358, symbol Amplifier_Operational:LM358
- added U9: MCP4725, Package_TO_SOT_SMD:SOT-23-6, symbol Analog_DAC:MCP4725xxx-xCH
Connections:
- net at C17.1, C18.1, C19.1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: now also K2.14, R16.2
- net GNDP: now reaches C14.2, C16.2, C17.2, C18.2, C19.2, C20.2, D2.2 (K), D2.3 (K), U6.1 (GND)
- net GNDP: now also K2.22, R11.2, R12.2
- net at U6.2 (FB): now also D3.2 (A), D4.2 (A), R15.2
- new net: C39.2, R35.1, U9.2 (-)
- new net: Q7.3 (C), R27.1, U9.3 (+)
- new net: C39.1, D10.1 (K), U9.6
- new net: C33.1, R32.2, U11.10 (+)
- new net: R22.1, R25.2, U11.8
- new net: R25.1, R26.1, U11.9 (-)
- new net: C10.2, R10.1, U2.2 (-)
- new net: K1.11, K1.21, K2.24, Q2.3 (S), R10.2, R18.2, R7.2
- new net: R45.1, R46.2, U11.5 (+)
- new net: C43.2, R41.2, U11.6 (-)
- new net: C43.1, R42.2, U11.7
- new net: Q8.1 (E), R23.1, R30.2
- new net: C35.1, C38.1, C42.1, Q10.3 (C), Q8.2 (C), R39.1
- new net: D10.2 (A), D11.2 (A), Q8.3 (B), R30.1, R34.2
- new net: C34.2, D11.1 (K), U10.6
- new net: C27.1, D3.1 (K), U7.1
- new net: C26.1, C27.2, R16.1, R17.1, U7.2 (-)
- new net: C28.1, D4.1 (K), U7.7
- new net: C9.1, R7.1, U2.5 (+)
- new net: R5.2, R6.2, U2.6 (-)
- new net: Q7.1 (B), R28.2
- new net: Q3.1 (B), R19.1
- new net: D5.2 (A), K2.A2, Q3.3 (C)
- new net: R29.2, U10.1 (VOUT)
- new net: Q1.1 (B), R8.1
- new net: C32.1, R31.2, U11.12 (+)
- new net: R31.1, R35.2, R39.2, R40.1
- new net: D1.2 (A), K1.A1, Q1.3 (C)
- new net: C10.1, R9.1, U2.1
- new net: Q10.2 (E), R38.1, R41.1
- new net: C34.1, R33.1, U10.2 (-)
- new net: R29.1, U10.3 (+)
- new net: K1.12, K1.22, R11.1
- new net: K1.14, K1.24, R12.1
- new net: J6.1 (Pin_1), K2.11
- new net: K2.12, Q2.2 (D)
- new net: J6.4 (Pin_4), K2.21
- new net: R21.1, U11.13 (-), U11.14
- new net: C28.2, R18.1, U7.6 (-)
- new net: Q10.1 (B), R42.1
- new net: Q2.1 (G), R9.2
- new net: R32.1, R33.2
- new net +12V: D1.1 (K), D5.1 (K), K1.A2, K2.A1
- new net +3V3: R45.2
- new net +3V3_DAC: C31.1, C32.1, C33.1, C34.1, R20.1, R25.1, U10.3 (VDD), U9.3 (VDD), U9.6 (A0)
- new net +5V: C24.1, C29.1, C37.1, C40.1, C7.1, R15.1, R34.1, U10.7 (V+), U11.4 (V+), U2.8 (V+), U7.8 (V+), U9.7 (V+)
- new net -5V: C25.1, C30.1, C36.1, C41.1, C8.1, U10.4 (V-), U11.11 (V-), U2.4 (V-), U7.4 (V-), U9.4 (V-)
- new net ADC_BOOST: C31.1, R23.2, R24.1
- new net ADC_DISCHARGE_CURRENT: R5.1, U2.7
- new net ADC_IOUT: D8.1 (K), R22.2
- new net ADC_VOUT: D9.1 (K), R21.2
- new net AGND: C31.2, C32.2, C33.2, R24.2, R26.2, R40.2
- new net CHRG_DISCH_MODE: R19.2
- new net DAC_CURRENT: U2.3 (+), U7.5 (+)
- new net DAC_OUT_VOLTAGE: R27.2, U9.1 (VOUT)
- new net DAC_VOLTAGE: U7.3 (+)
- new net DGND: C29.2, C30.2, C31.2, C32.2, C33.2, C34.2, C36.2, C37.2, C40.2, C41.2, D8.2 (A), D9.2 (A), Q7.2 (E), R46.1, U10.2 (VSS), U10.6 (A0), U9.2 (VSS)
- new net GND: C24.2, C25.2, C26.2, C7.2, C8.2, C9.2, Q1.2 (E), Q3.2 (E), R17.2, R6.1
- new net PGND: C35.2, C38.2, C42.2, R38.2
- new net SCL: R20.2, U10.5 (SCL), U9.5 (SCL)
- new net SDA: R25.2, U10.4 (SDA), U9.4 (SDA)
- new net SWITCH_METER: R28.1
- new net SWITCH_RANGE: R8.2
Other:
- note added: "CHARGE/DISCHARGE MODE SWITCH RELAY"
- note added: "CURRENT SET"
- note added: "CURRENT SOURCE"
- note added: "DISCHARGE CURRENT FEEDBACK TO ADC"
- note added: "DISCHARGE CURRENT RANGE SELECTOR"
- note added: "DISCHARGE CURRENT SOURCE REGULATOR"
- note added: "DUT VOLTAGE & CURRENT MEASURMRNT"
- note added: "VOLTAGE REGULATOR"
- note added: "VOLTAGE SET"
- moved on the sheet: C14, C15, C16, C17, C18, C19, C20, D2, L1, U6

Commit message: update charger schematic - voltage measurement
Parts:
- removed C29, C30, C32, C33: 100n, Capacitor_SMD:C_0805_2012Metric_Pad1.18x1.45mm_HandSolder, symbol Device:C
- removed D8, D9: LL4148, Diode_SMD:D_MiniMELF, symbol Diode:LL4148
- removed R21, R22: 470R, Resistor_SMD:R_0805_2012Metric_Pad1.20x1.40mm_HandSolder, symbol Device:R
- removed R25, R31, R32: 10k, Resistor_SMD:R_0805_2012Metric_Pad1.20x1.40mm_HandSolder, symbol Device:R
- removed R26: 1k, Resistor_SMD:R_0805_2012Metric_Pad1.20x1.40mm_HandSolder, symbol Device:R
- removed unit 3 of U11
- removed unit 5 of U11
- removed unit 4 of U11
- added C44, C45, C46: 100n, Capacitor_SMD:C_0805_2012Metric_Pad1.18x1.45mm_HandSolder, symbol Device:C
- added D12: 1N4148, Diode_THT:D_DO-35_SOD27_P7.62mm_Horizontal, symbol Diode:1N4148
- added D13, D14, D6, D7: D_Schottky, symbol Device:D_Schottky
- added K3: Relay_DPDT, symbol Relay:Relay_DPDT
- added Q4: BC817, Package_TO_SOT_SMD:SOT-23, symbol Transistor_BJT:BC817
- added R36, R37, R43, R44, R47, R48, R49, R50, R51: 10k, Capacitor_SMD:C_0805_2012Metric_Pad1.18x1.45mm_HandSolder, symbol Device:R
- added R52 (x2), R53 (x2), R54, R56: 10k/1%, Resistor_SMD:R_0805_2012Metric_Pad1.20x1.40mm_HandSolder, symbol Device:R
- added R57: 100R, Resistor_SMD:R_0805_2012Metric_Pad1.20x1.40mm_HandSolder, symbol Device:R
- added U12: LMV358, Package_SO:SOIC-8_3.9x4.9mm_P1.27mm, symbol Amplifier_Operational:LMV358
- added U13: INA128, symbol Amplifier_Instrumentation:INA128
Connections:
- net +12V: now also D12.1 (K), K3.A2, U13.7 (V+)
- net +5V: now also C46.1, U12.8 (V+)
- net -5V: now also C44.1, U13.4 (V-)
- net ADC_DISCHARGE_CURRENT: now also D13.2 (A), D14.1 (K), R51.2; no longer R5.1, U2.7
- net GND: now also C44.2, C45.2, C46.2, D14.2 (A), D7.2 (A), Q4.2 (E), R53.2, R54.2, U12.4 (V-)
- net at C17.1, C18.1, C19.1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: now also Q10.3 (C)
- net at C35.1, C38.1, C42.1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: no longer Q10.3 (C)
- net at J6.2 (Pin_2): now also R37.1
- net GND_VOLTAGE_DROP_INPUT: now reaches J6.3 (Pin_3)
- net GND_VOLTAGE_DROP_INPUT: now also R36.1, R52.2
- net SWITCH_RANGE renamed SWITCH_BATT_I_RANGE
- new net: K3.14, R49.1
- new net: Q4.1 (B), R48.1
- new net: D12.2 (A), K3.A1, Q4.3 (C)
- new net: R5.1, R51.1, U2.7
- new net: K3.11, R37.2, R44.1, U13.2 (-)
- new net: R43.1, U13.6
- new net: K3.24, R50.1
- new net: K3.21, R36.2, R47.1, U13.3 (+)
- new net: R56.1, R57.2, U12.7
- new net: R52.1, R53.1, U12.5 (+)
- new net: R53.2, U12.1, U12.2 (-)
- new net: R54.1, R56.2, U12.6 (-)
- new net: C45.1, R52.2, R53.1, U12.3 (+)
- new net ADC_BATT_VOLTAGE: D6.2 (A), D7.1 (K), R43.2
- new net GNDA: R44.2, R47.2, R49.2, R50.2, U13.5 (Ref)
- new net GND_VOLTAGE_DROP_ADC: R57.1
- new net SWITCH_BATT_V_RANGE: R48.2
- new net VREF_2V5: D13.1 (K), D6.1 (K), R52.1
Other:
- note added: "1,25V"
- note removed: "DUT VOLTAGE & CURRENT MEASURMRNT"
- moved on the sheet: C10, C14, C15, C16, C17, C18, C19, C20, C24, C25, C26, C27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

Commit message: update schematic
Parts:
- removed C31 (x2), C32, C36, C37, C40, C41, C42, C46: 100n, Capacitor_SMD:C_0805_2012Metric_Pad1.18x1.45mm_HandSolder, symbol Device:C
- removed C33, C34: 1u, Capacitor_SMD:C_0805_2012Metric_Pad1.18x1.45mm_HandSolder, symbol Device:C
- removed C34, C39: 100p, Capacitor_SMD:C_0805_2012Metric_Pad1.18x1.45mm_HandSolder, symbol Device:C
- removed C35: 220u/63V, Capacitor_THT:CP_Radial_D10.0mm_P5.00mm, symbol Device:C_Polarized
- removed C38: 10u/63V, Capacitor_SMD:C_1206_3216Metric, symbol Device:C
- removed D10, D11: LL4148, Diode_SMD:D_MiniMELF, symbol Diode:LL4148
- removed Q7: BC817, Package_TO_SOT_SMD:SOT-23, symbol Transistor_BJT:BC817
- removed Q8: BD136, Package_TO_SOT_THT:TO-126-3_Vertical, symbol Transistor_BJT:BD136
- removed R20, R23, R24, R25, R27, R28, R33: 10k, Resistor_SMD:R_0805_2012Metric_Pad1.20x1.40mm_HandSolder, symbol Device:R
- removed R29: 1K, Resistor_SMD:R_0805_2012Metric_Pad1.20x1.40mm_HandSolder, symbol Device:R
- removed R30: 2k7, Resistor_SMD:R_0805_2012Metric_Pad1.20x1.40mm_HandSolder, symbol Device:R
- removed R34, R35, R39, R40: 1k, Resistor_SMD:R_0805_2012Metric_Pad1.20x1.40mm_HandSolder, symbol Device:R
- removed U10: MCP4725xxx-xCH, Package_TO_SOT_SMD:SOT-23-6, symbol Analog_DAC:MCP4725xxx-xCH
- removed U10, U9: OP07, Package_SO:SO-8_3.9x4.9mm_P1.27mm, symbol Amplifier_Operational:OP07
- removed U11: LM324, Package_SO:SO-14_3.9x8.65mm_P1.27mm, symbol Amplifier_Operational:LM324
- removed U12: LMV358, Package_SO:SOIC-8_3.9x4.9mm_P1.27mm, symbol Amplifier_Operational:LMV358
- removed U9: MCP4725, Package_TO_SOT_SMD:SOT-23-6, symbol Analog_DAC:MCP4725xxx-xCH
- added C10, C13, C15, C16, C17: 100n, Capacitor_SMD:C_0805_2012Metric_Pad1.18x1.45mm_HandSolder, symbol Device:C
- added C11, C14: 1u, Capacitor_SMD:C_0805_2012Metric_Pad1.18x1.45mm_HandSolder, symbol Device:C
- added D1, D2: D_Schottky, symbol Device:D_Schottky
- added R10: 3k9, Capacitor_SMD:C_0805_2012Metric_Pad1.18x1.45mm_HandSolder, symbol Device:R
- added R11, R12: 1k, Capacitor_SMD:C_0805_2012Metric_Pad1.18x1.45mm_HandSolder, symbol Device:R
- added R13, R14: 100k, Capacitor_SMD:C_0805_2012Metric_Pad1.18x1.45mm_HandSolder, symbol Device:R
- added R2, R3, R7, R8: 56k, Capacitor_SMD:C_0805_2012Metric_Pad1.18x1.45mm_HandSolder, symbol Device:R
- added R9: 10k, Capacitor_SMD:C_0805_2012Metric_Pad1.18x1.45mm_HandSolder, symbol Device:R
- added U3, U6: MCP4725xxx-xCH, Package_TO_SOT_SMD:SOT-23-6, symbol Analog_DAC:MCP4725xxx-xCH
- added U7: LM324, symbol Amplifier_Operational:LM324
- renumbered C16 to C31, C14 to C32, C26 to C33, C15 to C34, C24 to C35, C25 to C36, C27 to C37, C28 to C38, C20 to C39, C19 to C40, C17 to C41, C18 to C42, C7 to C43, C8 to C44, C9 to C45, C10 to C46, C43 to C47, C44 to C48, C45 to C49, D5 to D10, D12 to D11, D6 to D12, D7 to D13, D3 to D4, D4 to D5, D2 to D6, D13 to D7, D14 to D8, D1 to D9, K1 to K2, K2 to K3, K3 to K4, Q1 to Q5, Q2 to Q6, Q10 to Q7, Q4 to Q8, Q3 to Q9, R17 to R28, R16 to R29, R18 to R30, R15 to R31, R51 to R32, R5 to R33, R6 to R34, R7 to R35, R8 to R36, R9 to R37, R10 to R38, R11 to R39, R12 to R40, R50 to R41, R49 to R42, R38 to R43, R37 to R44, R44 to R45, R19 to R46, R41 to R47, R36 to R48, R47 to R49, R42 to R50, R48 to R51, R45 to R52, R46 to R53, R43 to R54, R52 to R55, R53 to R56, R52 to R57, R53 to R58, R54 to R59, R56 to R60, R57 to R61, U7 to U11, U6 to U12, U2 to U13, U13 to U15
Connections:
- net +3V3 is gone; now on net VREF_2V5: R52.2
- net +5V: now also C15.1, U7.4 (V+)
- net -5V: now also C16.1, U7.11 (V-)
- net DAC_CURRENT: now also U6.1 (VOUT)
- net GND: now also C10.2, C11.2, C13.2, C14.2, C15.2, C16.2, C17.2, D2.2 (A), R11.1, U3.2 (VSS), U3.6 (A0), U6.2 (VSS), U6.6 (A0)
- net GND_VOLTAGE_DROP_INPUT: now also R14.2
- net SCL: now also R3.1, R8.1, U3.5 (SCL), U6.5 (SCL)
- net SDA: now also R2.1, R7.1, U3.4 (SDA), U6.4 (SDA)
- net VREF_2V5: now also D1.1 (K)
- net at R52.1, R53.2: now also U7.9 (-)
- net at C47.2, R47.2: now also U7.10 (+)
- net at C47.1, R50.2: now also U7.8
- net at J6.1 (Pin_1), K3.11: now also R13.1
- net at J6.4 (Pin_4), K3.21: now also R14.1
- net at R60.1, R61.2: now also U7.7
- net VBAT_INPUT: now reaches J6.2 (Pin_2), R44.1
- net VBAT_INPUT: now also R12.2, R13.2
- net at R57.1, R58.1: now also U7.6 (-)
- net at R58.2: now also U7.1, U7.2 (-)
- net at R59.1, R60.2: now also U7.5 (+)
- net at C49.1, R55.2, R56.1: now also U7.3 (+)
- net ADC_BATT_VOLTAGE renamed ADC_BATT_V_DIFF_OPAMP
- net DAC_VOLTAGE: no longer names the net of U11.3 (+)
- net DAC_VOLTAGE: now also U3.1 (VOUT)
- new net: R10.2, R11.2, U7.12 (+)
- new net: C17.1, R12.1, U7.13 (-)
- new net: R10.1, R9.1, U7.14
- new net +3.3V: C10.1, C11.1, C13.1, C14.1, R2.2, R3.2, R7.2, R8.2, U3.3 (VDD), U6.3 (VDD)
- new net ADC_CHARGE_VOLTAGE: D1.2 (A), D2.1 (K), R9.2
Other:
- note added: "12BIT I2C DAC FOR CURRENT REGULATION"
- note added: "12BIT I2C DAC FOR VOLTAGE REGULATION"
- note removed: "CURRENT SET"
- note removed: "CURRENT SOURCE"
- note removed: "VOLTAGE REGULATOR"
- note removed: "VOLTAGE SET"
- moved on the sheet: C31, C32, C34, C49, J6, R55, R56, R57, R58, R59, R60, R61
